File: elec/layout/default/rp2040.kicad_pcb (KiCad board)
At the start: 2 copper layers, 20 parts

Commit message: build with latest
Parts:
- C1, C2: value 20pF ±5% 50V C0G -> 22pF ±5% 50V C0G
- C10, C11, C3, C4, C5, C6, C7, C9: value 100nF ±10% 16V X7R -> 100nF ±10% 50V X7R
- C12, C8: value 1µF ±10% 16V X5R -> 1µF ±10% 25V X5R
Connections:
- U1 pad 13: sck-1 -> sck
- U1 pad 52: sck -> sck-1
- U3 pad 6: sck -> sck-1
Routing:
- net sck-1: track 0.00 -> 14.4 mm
- net sck: track 14.4 -> 0.00 mm
